Commit message: 电机多零位映射问题和电控已对接，readme增加了运行指令

File: src/tzb_description/urdf/tzb_description.urdf (robot description, URDF)
Before this commit: robot tzb_description, 11 links, 10 joints
Joints:
- joint J6_joint: limit lower=-2.8798 upper=2.8798 effort=3.5 velocity=2.0 -> lower=-3.14159 upper=3.14159 effort=3.5 velocity=2.0
- joint tcp_joint: origin xyz=-0.015 0.001 0.11 rpy=0 0 0 -> xyz=-0.02 -0.001 0.11 rpy=0 0 0
